File: Documents/kicad/headsetboard/ece445_headset.kicad_pcb (KiCad board)
At the start: 2 copper layers, 40 x 44.8 mm, 36 parts, among them J1 RCJ-054, J2 Conn_01x05_Female, J3 Screw_Terminal_01x02, J4 Conn_ARM_JTAG_SWD_10, Q1 SS8050-G, Q2 SS8050-G, SW1 SW_Push, SW2 SW_Push, U2 ESP32-S3-WROOM-1-N16R2, U3 AP2112K-3.3TRG1

Commit message: Add files via upload
Parts:
- removed H1, H2, H3, H4: MountingHole, MountingHole:MountingHole_3.2mm_M3
- removed JP3: SolderJumper_2_Open, Jumper:SolderJumper-2_P1.3mm_Open_TrianglePad1.0x1.5mm
- removed U3: AP2112K-3.3TRG1, csv_conn:SOT95P285X140-5N
- added U1: AP2112K-3.3TRG1, csv_conn:SOT95P285X140-5N, F.Cu at (154.3, 77.7)
- C2: value 1u -> 10u
- C3: value 1u -> 100n
- C4: value 10u -> 1u
- C5: value 100n -> 1u
- JP2: value SolderJumper_3_Open -> SolderJumper_2_Open; footprint Jumper:SolderJumper-3_P2.0mm_Open_TrianglePad1.0x1.5mm -> Jumper:SolderJumper-2_P1.3mm_Open_TrianglePad1.0x1.5mm
- R1: value 1k -> 10k
- R3: value 10k -> 1k
- U2: value ESP32-S3-WROOM-1-N16R2 -> ESP32-WROVER-E-N4R8; footprint local_footprints:ESP32-S3-WROOM-1_EXP -> csv_conn:ESP32­WROVER­E&slash_ESP32­WROVER­IE_EXP
- moved R4 91.7 mm to (169.0, 72.5), turned to -90 degrees
- moved C5 84.6 mm to (166.5, 72.5)
- moved JP2 84.0 mm to (156.3, 86.0), turned to 0 degrees
- moved C9 81.6 mm to (158.5, 82.0), turned to 180 degrees
- moved C8 78.5 mm to (158.5, 78.5), turned to 180 degrees
- moved R3 77.6 mm to (171.5, 72.5), turned to -90 degrees
- moved C2 76.3 mm to (147.5, 79.5), turned to -90 degrees
- moved R1 75.1 mm to (152.5, 73.5)
- moved TP1 74.3 mm to (151.5, 85.0)
- moved R8 74.0 mm to (164.0, 72.5), turned to 90 degrees
- moved U2 72.5 mm to (163.3, 52.8)
- moved R6 72.2 mm to (161.5, 72.6), turned to 90 degrees
- moved C6 72.1 mm to (151.0, 45.5)
- moved C7 72.1 mm to (148.0, 45.5)
- moved SW2 71.4 mm to (167.5, 79.5), turned to 0 degrees
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Connections:
- net /GPIO15 renamed /GPIO32
- net /GPIO16 renamed /GPIO33
- net /GPIO5 renamed /SENSOR_VN
- net /GPIO6 renamed /GPIO34
- net /GPIO7 renamed /GPIO35
- net /GPIO8 renamed /GPIO27
- C2 pad 1: /CHIP_PU -> +BATT
- C3 pad 1: /GPIO0_STRAPPING -> +BATT
- C4 pad 1: +BATT -> /CHIP_PU
- C5 pad 1: +BATT -> /GPIO0_STRAPPING
- C8 pad 1: Net-(JP3-A) -> Net-(JP2-A)
- C9 pad 1: Net-(JP3-A) -> Net-(JP2-A)
- J1 pad 2: /CSV_OUT -> /DAC1_OUT
- JP2 pad 1: GND -> Net-(JP2-A)
- JP2 pad 2: Net-(JP2-C) -> +3V3
- R1 pad 1: /GPIO46_STRAPPING -> /DTR
- R1 pad 2: +3V3 -> Net-(Q1-B)
- R2 pad 1: /DTR -> /RTS
- R2 pad 2: Net-(Q1-B) -> Net-(Q2-B)
- R3 pad 1: /RTS -> /GPIO2_STRAPPING
- R3 pad 2: Net-(Q2-B) -> +3V3
- R4 pad 1: /GPIO3_STRAPPING -> /GPIO5_STRAPPING
- R4 pad 2: Net-(JP2-C) -> GND
- TP1 pad 1: Net-(JP3-A) -> Net-(JP2-A)
- U2 pad 10: /GPIO17 -> /DAC1_OUT
- U2 pad 11: /GPIO18 -> /GPIO26
- U2 pad 13: /GPIO19 -> /MTMS
- U2 pad 14: /GPIO20 -> /MTDI
- U2 pad 15: /GPIO3_STRAPPING -> GND
- U2 pad 16: /GPIO46_STRAPPING -> /MTCK
- U2 pad 17: /GPIO9 -> unconnected-(U2-NC-Pad17)
- U2 pad 18: /GPIO10 -> unconnected-(U2-NC-Pad18)
- U2 pad 19: /GPIO11 -> unconnected-(U2-NC-Pad19)
- U2 pad 20: /GPIO12 -> unconnected-(U2-NC-Pad20)
- U2 pad 21: /GPIO21 -> unconnected-(U2-NC-Pad21)
- U2 pad 22: /GPIO14 -> unconnected-(U2-NC-Pad22)
- U2 pad 23: /GPIO23 -> /MTDO
- U2 pad 24: /GPIO24 -> /GPIO2_STRAPPING
- U2 pad 25: /GPIO48 -> /GPIO0_STRAPPING
- U2 pad 26: /GPIO45_STRAPPING -> /GPIO4
- U2 pad 27: /GPIO0_STRAPPING -> unconnected-(U2-NC-Pad27)
- U2 pad 28: /GPIO28 -> unconnected-(U2-NC-Pad28)
- U2 pad 29: /GPIO29 -> /GPIO5_STRAPPING
- U2 pad 30: /GPIO37 -> /GPIO18
- U2 pad 31: /GPIO38 -> /GPIO19
- U2 pad 32: /MTCK -> unconnected-(U2-NC-Pad32)
- U2 pad 33: /MTDO -> /GPIO21
- U2 pad 34: /MTDI -> /RX
- U2 pad 35: /MTMS -> /TX
- U2 pad 36: /RX -> /GPIO22
- U2 pad 37: /TX -> /GPIO23
- U2 pad 38: /CSV_OUT -> GND
- U2 pad 39: /GPIO1 -> GND
- U2 pad 4: /GPIO4 -> /SENSOR_VP
Routing:
- net /CHIP_PU: track 81.4 -> 56.3 mm, vias 2 -> 0
- net Net-(JP2-A): track 0.00 -> 21.8 mm
- net /GPIO5_STRAPPING: track 0.00 -> 18.6 mm, vias 0 -> 2
- net /MTDO: track 17.9 -> 35.1 mm, vias 0 -> 2
- net Net-(JP3-A): track 16.0 -> 0.00 mm
- net /RTS: track 12.0 -> 25.9 mm
- net /GPIO0_STRAPPING: track 24.0 -> 37.7 mm
- net /GPIO2_STRAPPING: track 0.00 -> 11.8 mm
- net /CSV_OUT: track 8.72 -> 0.00 mm
- net /GPIO46_STRAPPING: track 8.51 -> 0.00 mm
- net +BATT: track 28.1 -> 19.8 mm
- net /MTMS: track 25.1 -> 17.1 mm, vias 2 -> 0
- net +3V3: track 100.0 -> 92.5 mm, vias 5 -> 7
- net /DAC1_OUT: track 0.00 -> 7.51 mm
- net /MTDI: track 17.7 -> 24.7 mm
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Other:
- board size 40 x 44.8 mm -> 42.5 x 44.5 mm
