File: Documents/kicad/headsetboard/ece445_headset.kicad_sch (KiCad schematic)
At the start: 48 parts, among them J1 Screw_Terminal_01x02, J2 Conn_01x05_Female, J3 Conn_ARM_JTAG_SWD_10, Q1 AO4485, Q2 SS8050-G, Q3 SS8050-G, SW1 SW_Push, SW2 SW_Push, U1 TPS62933ODRLR, U2 ESP32-S3-WROOM-1-N16R2

Commit message: Add files via upload
Parts:
- added J4: PJRAN1X1U04X, csv_conn:SWITCHCRAFT_PJRAN1X1U04X, symbol csv_conn:PJRAN1X1U04X
Connections:
- net GND: now also J4.2, J4.3
- net GPIO2 renamed CSV_OUT
- net CSV_OUT: now also J4.1

Commit message: Add files via upload
Parts:
- removed C8: 100n, Capacitor_SMD:C_0805_2012Metric, symbol basic:C
- removed D1: D_Zener, local_footprints:SOD-123_ONS, symbol Device:D_Zener
- removed F1: Fuse, Fuse:Fuseholder_Littelfuse_Nano2_154x, symbol Device:Fuse
- removed J4: PJRAN1X1U04X, csv_conn:SWITCHCRAFT_PJRAN1X1U04X, symbol csv_conn:PJRAN1X1U04X
- removed L1: 4.7u, Inductor_SMD:L_Taiyo-Yuden_NR-60xx, symbol basic:L
- removed Q1: AO4485, local_footprints:SO8SOP-8L_AOS, symbol local_symbols:AO4485
- removed R1, R13: 100k, Resistor_SMD:R_0805_2012Metric, symbol basic:R
- removed R12, R8, R9: DNP, Resistor_SMD:R_0805_2012Metric, symbol basic:R
- removed R14: 31.3k, Resistor_SMD:R_0805_2012Metric, symbol basic:R
- removed R15: 10.0k, Resistor_SMD:R_0805_2012Metric, symbol basic:R
- removed TP1: TestPoint, TestPoint:TestPoint_Pad_D2.0mm, symbol Connector:TestPoint
- removed U1: TPS62933ODRLR, local_footprints:SOT5X3-8_DRL_TEX, symbol local_symbols:TPS62933ODRLR
- added J1: RCJ-054, csv_conn:CUI_RCJ-054, symbol csv_conn:RCJ-054
- added U3: AP2112K-3.3TRG1, csv_conn:SOT95P285X140-5N, symbol ldo:AP2112K-3.3TRG1
- renumbered C9 to C8, C10 to C9, J1 to J3, J3 to J4, Q2 to Q1, Q3 to Q2, R2 to R1, R3 to R2, R4 to R3, R5 to R4, R6 to R5, R7 to R6, R10 to R7, R11 to R8, TP2 to TP1, TP3 to TP2
Connections:
- net +BATT: now also J3.2 (Pin_2), U3.1 (VIN), U3.3 (EN)
- net CSV_OUT: now also J1.2
- net GND: now also J1.1, U3.2 (GND)
- net at C8.1, C9.1, JP3.1 (A)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: now also U3.5 (VOUT)
Other:
- note added: "Battery Input"
- note removed: "Battery Input and RVP"
- moved on the sheet: C1, C4, C5, C8, C9, J3, JP3, TP1, TP2

Commit message: Add files via upload
Parts:
- removed H1, H2, H3, H4: MountingHole, MountingHole:MountingHole_3.2mm_M3, symbol Mechanical:MountingHole
- removed JP2: SolderJumper_3_Open, Jumper:SolderJumper-3_P2.0mm_Open_TrianglePad1.0x1.5mm, symbol Jumper:SolderJumper_3_Open
- removed R1: 1k, Resistor_SMD:R_0805_2012Metric, symbol basic:R
- removed U2: ESP32-S3-WROOM-1-N16R2, local_footprints:ESP32-S3-WROOM-1_EXP, symbol local_symbols:ESP32-S3-WROOM-1-N16R2
- added R3: 1k, Resistor_SMD:R_0805_2012Metric, symbol basic:R
- added U2: ESP32-WROVER-E-N4R8, csv_conn:ESP32­WROVER­E&slash_ESP32­WROVER­IE_EXP, symbol esp:ESP32-WROVER-E-N4R8
- R4: Note (none) -> DNP
- renumbered C4 to C2, C5 to C3, C2 to C4, C3 to C5, JP3 to JP2, R2 to R1, R3 to R2, U3 to U1
Connections:
- net +3V3: now also R3.2, U2.2 (3V3)
- net CHIP_PU: now also U2.3 (EN)
- net GND: now also R4.2, U2.1 (GND), U2.15 (GND), U2.38 (GND), U2.39 (GND), U2.40 (GND), U2.41 (GND), U2.42 (GND), U2.43 (GND), U2.44 (GND), U2.45 (GND), U2.46 (GND), U2.47 (GND)
- net GPIO0_STRAPPING: now also U2.25 (IO0)
- net GPIO18: now also U2.30 (IO18)
- net GPIO19: now also U2.31 (IO19)
- net GPIO21: now also U2.33 (IO21)
- net GPIO23: now also U2.37 (IO23)
- net GPIO4: now also U2.26 (IO4)
- net MTCK: now also U2.16 (IO13)
- net MTDI: now also U2.14 (IO12)
- net MTDO: now also U2.23 (IO15)
- net MTMS: now also U2.13 (IO14)
- net RX: now also U2.34 (RXD0)
- net TX: now also U2.35 (TXD0)
- net CSV_OUT renamed DAC1_OUT
- net DAC1_OUT: now also U2.10 (IO25)
- net GPIO3_STRAPPING renamed GPIO5_STRAPPING
- net GPIO5_STRAPPING: now also U2.29 (IO5)
- new net GPIO22: U2.36 (IO22)
- new net GPIO26: U2.11 (IO26)
- new net GPIO27: U2.12 (IO27)
- new net GPIO2_STRAPPING: R3.1, U2.24 (IO2)
- new net GPIO32: U2.8 (IO32)
- new net GPIO33: U2.9 (IO33)
- new net GPIO34: U2.6 (IO34)
- new net GPIO35: U2.7 (IO35)
- new net SENSOR_VN: U2.5 (SENSOR_VN)
- new net SENSOR_VP: U2.4 (SENSOR_VP)
Other:
- note removed: "Mounting Holes"
