File: Documents/kicad/adapter_board/adapter_board/adapter_board.kicad_pcb (KiCad board)
At the start: 2 copper layers, 2 parts

Commit message: new stuff
Parts:
- removed VAL** (x2): CF2-DECK-SMD-HOLES, libs:CF2-DECK-SMD-HOLES
- added REF**: Connector_Crazyflie, footprints_crazyflie_connector:CONN10X1_NPPN101BFLC-RC_SUL, F.Cu at (155.0, 70.0)
- added REF**: Connector_Crazyflie, footprints_crazyflie_connector:CONN10X1_NPPN101BFLC-RC_SUL, F.Cu at (155.0, 45.0)
- added REF**: Connector_ESPCam, footprints_espcam_connector:CONN_NPTC081KFXC-RC_SUL, B.Cu at (155.0, 68.9)
- added REF**: Connector_ESPCam, footprints_espcam_connector:CONN_NPTC081KFXC-RC_SUL, B.Cu at (155.0, 46.0)
Other:
- board text added: "Antenna"
- board text added: "Back CrazyFlie"
- board text added: "Front CrazyFlie"
- board text added: "No Antenna"

Commit message: schematic finished
Parts:
- removed REF** (x2): Connector_Crazyflie, footprints_crazyflie_connector:CONN10X1_NPPN101BFLC-RC_SUL
- removed REF** (x2): Connector_ESPCam, footprints_espcam_connector:CONN_NPTC081KFXC-RC_SUL
- added J3: Crazyflie Right, footprints_crazyflie_connector:CONN10X1_NPPN101BFLC-RC_SUL, F.Cu at (65.4, 61.9)
- added TP1: Vout LDO, TestPoint:TestPoint_THTPad_1.5x1.5mm_Drill0.7mm, F.Cu at (78.4, 59.1)
Other:
- board text removed: "Antenna"
- board text removed: "Back CrazyFlie"
- board text removed: "Front CrazyFlie"
- board text removed: "No Antenna"

Commit message: finished board
Parts:
- added C1: 10u, Capacitor_SMD:C_0805_2012Metric_Pad1.18x1.45mm_HandSolder, F.Cu at (159.9, 70.2)
- added C2: 10u, Capacitor_SMD:C_0805_2012Metric_Pad1.18x1.45mm_HandSolder, F.Cu at (159.9, 73.2)
- added C3: 10u, Capacitor_SMD:C_0805_2012Metric_Pad1.18x1.45mm_HandSolder, F.Cu at (159.9, 76.2)
- added C4: 33u, Capacitor_SMD:C_0805_2012Metric_Pad1.18x1.45mm_HandSolder, F.Cu at (165.4, 73.0)
- added C5: 33u, Capacitor_SMD:C_0805_2012Metric_Pad1.18x1.45mm_HandSolder, F.Cu at (165.4, 76.0)
- added J1: ESP Cam Left, footprints_espcam_connector:CONN_NPTC081KFXC-RC_SUL, B.Cu at (165.0, 82.9)
- added J2: Crazyflie Left, footprints_crazyflie_connector:CONN10X1_NPPN101BFLC-RC_SUL, F.Cu at (165.0, 82.0)
- added J4: ESP Cam Right, footprints_espcam_connector:CONN_NPTC081KFXC-RC_SUL, B.Cu at (165.0, 60.0)
- added JP1: Jumper, Jumper:SolderJumper-2_P1.3mm_Open_TrianglePad1.0x1.5mm, F.Cu at (164.1, 65.8)
- added U1: AP2112K-3.3TRG1, footprints:SOT95P285X140-5N, F.Cu at (170.4, 73.7)
- moved J3 99.6 mm to (165.0, 60.0)
- moved TP1 92.2 mm to (170.3, 67.5)
Connections:
- J3 pad 9: /VCOM -> /LDO_IN
Routing:
- net /LDO_IN: track 0.00 -> 40.2 mm, vias 0 -> 2
- net Net-(JP1-A): track 0.00 -> 31.7 mm
- net /3v3: track 0.00 -> 14.0 mm, vias 0 -> 1
- net GND: vias 0 -> 7
- added copper zone on B.Cu, net GND
- added copper zone on F.Cu, net GND
Other:
- board outline added: 25 x 31.3 mm
- board text added: "Crazyflie Antenna"
- board text added: "Crazyflie Rear"
- board text added: "ECE445 SP24 Adapter Board Hunter Baisden Team 64"
- board text added: "ESP32 Cam Back"
- board text added: "ESP32 Cam Front"

Commit message: adding gerber files
Other:
- board text added: "ECE445 SP24 Adapter Board Team 64 Hunter Baisden"
- board text removed: "ECE445 SP24 Adapter Board Hunter Baisden Team 64"
Changed lines of the file:
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@@
 		(layer "Edge.Cuts")
 	)
-	(gr_text "ECE445 SP24 \nAdapter Board\nHunter Baisden Team 64"
-		(at 172.38 73.42 0)
+	(gr_text "ECE445 SP24 \nAdapter Board\nTeam 64\nHunter Baisden"
+		(at 165.3925 75.96 0)
 		(layer "B.SilkS")
 		(effects
@@
 				(thickness 0.15)
 			)
-			(justify left bottom mirror)
+			(justify bottom mirror)
 		)
 	)
 	(gr_text "ESP32 Cam Front"
-		(at 156.37 64.51 90)
+		(at 155.04 64.32 90)
 		(layer "B.SilkS")
 		(effects
@@
 	)
 	(gr_text "Crazyflie Antenna"
-		(at 156.19 77.36 90)
+		(at 155.04 77.46 90)
 		(layer "F.SilkS")
 		(effects
